File: ledboard/segment_led.kicad_sch (KiCad schematic)
At the start: 11 parts, among them U6 TBD62083AFG, U7 TBD62783AFG

Commit message: 各種定数見直し,TPS2121の前後にデカップリングコンデンサを配置.
Parts:
- U6: MPN TBF62083AFG -> TBD62083AFG
Changed lines of the file:
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@@
+	)
+	(symbol
+		(lib_id "MyLib:TBD62083AFG")
+		(at 106.68 59.69 0)
+		(unit 1)
+		(exclude_from_sim no)
+		(in_bom yes)
+		(on_board yes)
+		(dnp no)
+		(fields_autoplaced yes)
+		(property "Reference" "U6"
+			(at 106.68 45.72 0)
+			(effects
+				(font
+					(size 1.524 1.524)
+				)
+			)
+		)
+		(property "Value" "TBD62083AFG"
+			(at 106.68 48.26 0)
+			(effects
+				(font
+					(size 1.524 1.524)
+				)
+			)
+		)
+		(property "Footprint" "MyLib:SOP18-P-375-1p27_TOS"
+			(at 107.188 81.28 0)
+			(effects
+				(font
+					(size 1.27 1.27)
+					(italic yes)
+				)
+				(hide yes)
+			)
+		)
+		(property "Datasheet" "https://toshiba.semicon-storage.com/info/docget.jsp?did=29808&prodName=TBD62083AFG"
+			(at 113.538 84.328 0)
+			(effects
+				(font
+					(size 1.27 1.27)
+					(italic yes)
+				)
+				(hide yes)
+			)
+		)
+		(property "Description" ""
+			(at 106.68 59.69 0)
+			(effects
+				(font
+					(size 1.27 1.27)
+				)
+				(hide yes)
+			)
+		)
+		(property "Manufacturer" "Toshiba"
+			(at 105.918 90.678 0)
+			(effects
+				(font
+					(size 1.27 1.27)
+				)
+				(hide yes)
+			)
+		)
+		(property "MPN" "TBD62083AFG"
+			(at 107.188 87.63 0)
+			(effects
+				(font
+					(size 1.27 1.27)
+				)
+				(hide yes)
+			)
+		)
+		(pin "4"
+		)
+		(pin "6"
+		)
+		(pin "5"
+		)
+		(pin "14"
+		)
+		(pin "15"
+		)
+		(pin "18"
+		)
+		(pin "3"
+		)
+		(pin "16"
+		)
+		(pin "12"
+		)
+		(pin "9"
+		)
+		(pin "8"
+		)
+		(pin "10"
+		)
+		(pin "17"
+		)
+		(pin "13"
+		)
+		(pin "7"
+		)
+		(pin "11"
+		)
+		(pin "2"
+		)
+		(pin "1"
+		)
+		(instances
+			(project "ledboard"
+				(path "/bdb2205c-1d8b-445a-876a-0efe4f06b647/a778b9b9-a786-4f14-8ba2-902f86c2e4ab"
+					(reference "U6")
+					(unit 1)
+				)
+			)
+		)
 	)
 	(symbol
@@
 					(unit 1)
 				)
-			)
-		)
-	)
-	(symbol
-		(lib_id "MyLib:TBD62083AFG")
-		(at 106.68 59.69 0)
-		(unit 1)
-		(exclude_from_sim no)
-		(in_bom yes)
-		(on_board yes)
-		(dnp no)
-		(fields_autoplaced yes)
-		(property "Reference" "U6"
-			(at 106.68 45.72 0)
-			(effects
-				(font
-					(size 1.524 1.524)
-				)
-			)
-		)
-		(property "Value" "TBD62083AFG"
-			(at 106.68 48.26 0)
-			(effects
-				(font
-					(size 1.524 1.524)
-				)
-			)
-		)
-		(property "Footprint" "MyLib:SOP18-P-375-1p27_TOS"
-			(at 107.188 81.28 0)
-			(effects
-				(font
-					(size 1.27 1.27)
-					(italic yes)
-				)
-				(hide yes)
-			)
-		)
-		(property "Datasheet" "https://toshiba.semicon-storage.com/info/docget.jsp?did=29808&prodName=TBD62083AFG"
-			(at 113.538 84.328 0)
-			(effects
-				(font
-					(size 1.27 1.27)
-					(italic yes)
-				)
-				(hide yes)
-			)
-		)
-		(property "Description" ""
-			(at 106.68 59.69 0)
-			(effects
-				(font
-					(size 1.27 1.27)
-				)
-				(hide yes)
-			)
-		)
-		(property "Manufacturer" "Toshiba"
-			(at 105.918 90.678 0)
-			(effects
-				(font
-					(size 1.27 1.27)
-				)
-				(hide yes)
-			)
-		)
-		(property "MPN" "TBF62083AFG"
-			(at 107.188 87.63 0)
-			(effects
-				(font
-					(size 1.27 1.27)
-				)
-				(hide yes)
-			)
-		)
-		(pin "8"
-		)
-		(pin "18"
-		)
-		(pin "3"
-		)
-		(pin "7"
-		)
-		(pin "6"
-		)
-		(pin "16"
-		)
-		(pin "14"
-		)
-		(pin "5"
-		)
-		(pin "2"
-		)
-		(pin "1"
-		)
-		(pin "10"
-		)
-		(pin "17"
-		)
-		(pin "4"
-		)
-		(pin "11"
-		)
-		(pin "15"
-		)
-		(pin "12"
-		)
-		(pin "13"
-		)
-		(pin "9"
-		)
-		(instances
-			(project "ledboard"
-				(path "/bdb2205c-1d8b-445a-876a-0efe4f06b647/a778b9b9-a786-4f14-8ba2-902f86c2e4ab"
-					(reference "U6")
-					(unit 1)
-				)

Commit message: 部品の再アノテーションを行う.
Parts:
- renumbered R29 to R33, R30 to R34, R31 to R35, R32 to R36, R33 to R37, R34 to R38, R35 to R39, R36 to R40, U6 to U7, U7 to U8
Changed lines of the file:
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@@
 		(dnp no)
 		(fields_autoplaced yes)
-		(property "Reference" "R32"
+		(property "Reference" "R36"
 			(at 154.94 100.33 90)
 			(effects
@@
 			(project "ledboard"
 				(path "/bdb2205c-1d8b-445a-876a-0efe4f06b647/a778b9b9-a786-4f14-8ba2-902f86c2e4ab"
-					(reference "R32")
+					(reference "R36")
 					(unit 1)
 				)
@@
 		(dnp no)
 		(fields_autoplaced yes)
-		(property "Reference" "R29"
+		(property "Reference" "R33"
 			(at 132.08 92.71 90)
 			(effects
@@
 			(project "ledboard"
 				(path "/bdb2205c-1d8b-445a-876a-0efe4f06b647/a778b9b9-a786-4f14-8ba2-902f86c2e4ab"
-					(reference "R29")
+					(reference "R33")
 					(unit 1)
 				)
@@
 		(dnp no)
 		(fields_autoplaced yes)
-		(property "Reference" "U7"
+		(property "Reference" "U8"
 			(at 107.95 88.9 0)
 			(effects
@@
 			(project "ledboard"
 				(path "/bdb2205c-1d8b-445a-876a-0efe4f06b647/a778b9b9-a786-4f14-8ba2-902f86c2e4ab"
-					(reference "U7")
+					(reference "U8")
 					(unit 1)
 				)
@@
 		(dnp no)
 		(fields_autoplaced yes)
-		(property "Reference" "R36"
+		(property "Reference" "R40"
 			(at 185.42 110.49 90)
 			(effects
@@
 			(project "ledboard"
 				(path "/bdb2205c-1d8b-445a-876a-0efe4f06b647/a778b9b9-a786-4f14-8ba2-902f86c2e4ab"
-					(reference "R36")
+					(reference "R40")
 					(unit 1)
 				)
@@
 		(dnp no)
 		(fields_autoplaced yes)
-		(property "Reference" "R31"
+		(property "Reference" "R35"
 			(at 147.32 97.79 90)
 			(effects
@@
 			(project "ledboard"
 				(path "/bdb2205c-1d8b-445a-876a-0efe4f06b647/a778b9b9-a786-4f14-8ba2-902f86c2e4ab"
-					(reference "R31")
+					(reference "R35")
 					(unit 1)
 				)
@@
 		(dnp no)
 		(fields_autoplaced yes)
-		(property "Reference" "R33"
+		(property "Reference" "R37"
 			(at 162.56 102.87 90)
 			(effects
@@
 			(project "ledboard"
 				(path "/bdb2205c-1d8b-445a-876a-0efe4f06b647/a778b9b9-a786-4f14-8ba2-902f86c2e4ab"
-					(reference "R33")
+					(reference "R37")
 					(unit 1)
 				)
@@
 		(dnp no)
 		(fields_autoplaced yes)
-		(property "Reference" "U6"
+		(property "Reference" "U7"
 			(at 106.68 45.72 0)
 			(effects
@@
 			(project "ledboard"
 				(path "/bdb2205c-1d8b-445a-876a-0efe4f06b647/a778b9b9-a786-4f14-8ba2-902f86c2e4ab"
-					(reference "U6")
+					(reference "U7")
 					(unit 1)
 				)
@@
 		(dnp no)
 		(fields_autoplaced yes)
-		(property "Reference" "R35"
+		(property "Reference" "R39"
 			(at 177.8 107.95 90)
 			(effects
@@
 			(project "ledboard"
 				(path "/bdb2205c-1d8b-445a-876a-0efe4f06b647/a778b9b9-a786-4f14-8ba2-902f86c2e4ab"
-					(reference "R35")
+					(reference "R39")
 					(unit 1)
 				)
@@
 		(dnp no)
 		(fields_autoplaced yes)
-		(property "Reference" "#PWR014"
+		(property "Reference" "#PWR018"
 			(at 87.63 86.36 0)
 			(effects
@@
 			(project "ledboard"
 				(path "/bdb2205c-1d8b-445a-876a-0efe4f06b647/a778b9b9-a786-4f14-8ba2-902f86c2e4ab"
-					(reference "#PWR014")
+					(reference "#PWR018")
 					(unit 1)
 				)
@@
 		(dnp no)
 		(fields_autoplaced yes)
-		(property "Reference" "R34"
+		(property "Reference" "R38"
 			(at 170.18 105.41 90)
 			(effects
@@
 			(project "ledboard"
 				(path "/bdb2205c-1d8b-445a-876a-0efe4f06b647/a778b9b9-a786-4f14-8ba2-902f86c2e4ab"
-					(reference "R34")
+					(reference "R38")
 					(unit 1)
 				)
@@
 		(dnp no)
 		(fields_autoplaced yes)
-		(property "Reference" "R30"
+		(property "Reference" "R34"
 			(at 139.7 95.25 90)
 			(effects
@@
 			(project "ledboard"
 				(path "/bdb2205c-1d8b-445a-876a-0efe4f06b647/a778b9b9-a786-4f14-8ba2-902f86c2e4ab"
-					(reference "R30")
+					(reference "R34")
 					(unit 1)
 				)
@@
 		(dnp no)
 		(fields_autoplaced yes)
-		(property "Reference" "#PWR016"
+		(property "Reference" "#PWR019"
 			(at 127 132.08 0)
 			(effects
@@
 			(project "ledboard"
 				(path "/bdb2205c-1d8b-445a-876a-0efe4f06b647/a778b9b9-a786-4f14-8ba2-902f86c2e4ab"
-					(reference "#PWR016")
-					(unit 1)
-				)
+					(reference "#PWR019")
+					(unit 1)
+				)

Commit message: 部品が決まったので,コミットします.
Parts:
- D11: renamed from L3; footprint (none) -> MyLib:SN620362B; MPN (none) -> SN620362B; Manufacturer (none) -> ARKLED
- R33, R34, R35, R36, R37, R38, R39, R40: value 62 -> 100; footprint (none) -> Resistor_SMD:R_0603_1608Metric; MPN (none) -> SR0603FR-7T100RL; Manufacturer (none) -> YAGEO
- U8: MPN (none) -> TBD62783AFG; Manufacturer (none) -> Toshiba
Connections:
- net +5V renamed +5V_VCC
Other:
- note added: "7 Segment LED"

Commit message: LSCS品番を追加. コンデンサの品番を変更します.
Parts:
- D11: LCSC Part # (none) -> C96556
- R33, R34, R35, R36, R37, R38, R39, R40: LCSC Part # (none) -> C873671
- U7: LCSC Part # (none) -> C163228
- U8: LCSC Part # (none) -> C97745
Changed lines of the file:
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@@
 	(generator_version "9.0")
 	(paper "A4")
+	(title_block
+		(date "2026-04-15")
+		(rev "1.0")
+	)
 	(text "7 Segment LED"
 		(exclude_from_sim no)
@@
 			)
 		)
+		(property "LCSC Part #" "C873671"
+			(at 154.94 106.68 90)
+			(effects
+				(font
+					(size 1.27 1.27)
+				)
+				(hide yes)
+			)
+		)
 		(pin "1"
 		)
@@
 			)
 		)
+		(property "LCSC Part #" "C873671"
+			(at 132.08 99.06 90)
+			(effects
+				(font
+					(size 1.27 1.27)
+				)
+				(hide yes)
+			)
+		)
 		(pin "1"
 		)
@@
 			)
 		)
+		(property "LCSC Part #" "C97745"
+			(at 87.63 99.06 0)
+			(effects
+				(font
+					(size 1.27 1.27)
+				)
+				(hide yes)
+			)
+		)
 		(pin "11"
 		)
@@
 			)
 		)
+		(property "LCSC Part #" "C873671"
+			(at 185.42 116.84 90)
+			(effects
+				(font
+					(size 1.27 1.27)
+				)
+				(hide yes)
+			)
+		)
 		(pin "1"
 		)
@@
 			)
 		)
+		(property "LCSC Part #" "C873671"
+			(at 147.32 104.14 90)
+			(effects
+				(font
+					(size 1.27 1.27)
+				)
+				(hide yes)
+			)
+		)
 		(pin "1"
 		)
@@
 			)
 		)
+		(property "LCSC Part #" "C873671"
+			(at 162.56 109.22 90)
+			(effects
+				(font
+					(size 1.27 1.27)
+				)
+				(hide yes)
+			)
+		)
 		(pin "1"
 		)
@@
 			)
 		)
+		(property "LCSC Part #" "C163228"
+			(at 106.68 59.69 0)
+			(effects
+				(font
+					(size 1.27 1.27)
+				)
+				(hide yes)
+			)
+		)
 		(pin "4"
 		)
@@
 			)
 		)
+		(property "LCSC Part #" "C873671"
+			(at 177.8 114.3 90)
+			(effects
+				(font
+					(size 1.27 1.27)
+				)
+				(hide yes)
+			)
+		)
 		(pin "1"
 		)
@@
 			)
 		)
+		(property "LCSC Part #" "C873671"
+			(at 170.18 111.76 90)
+			(effects
+				(font
+					(size 1.27 1.27)
+				)
+				(hide yes)
+			)
+		)
 		(pin "1"
 		)
@@
 		)
 		(property "Manufacturer" "ARKLED"
+			(at 214.63 90.17 0)
+			(effects
+				(font
+					(size 1.27 1.27)
+				)
+				(hide yes)
+			)
+		)
+		(property "LCSC Part #" "C96556"
 			(at 214.63 90.17 0)
 			(effects
@@
 			(at 139.7 101.6 90)
 			(effects
+				(font
+					(size 1.27 1.27)
+				)
+				(hide yes)
+			)
+		)
+		(property "LCSC Part #" "C873671"
+			(at 139.7 101.6 90)
+			(effects
